File: opto_elec_boards/phd_slave/phd_slave.kicad_pcb (KiCad board)
At the start: 2 copper layers, 63 x 95.2 mm, 20 parts, among them J1 From Main Board, M4a MountingHole_4.3mm_M4, M4b MountingHole_4.3mm_M4, M4c MountingHole_4.3mm_M4, M4d MountingHole_4.3mm_M4, U1 TL082, U2 OPA551

Commit message: Update Opto Boards / To change : var +15V and var -15V ?
Other:
- board text added: "+15V"
- board text added: "IN1"
Changed lines of the file:
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@@
 		(tags "Through hole angled socket strip THT 2x10 2.54mm double row")
 		(property "Reference" "J1"
-			(at -5.65 -2.77 0)
+			(at -7.79 -3.25 90)
 			(layer "F.SilkS")
 			(effects
@@
 		)
 	)
+	(gr_text "+15V"
+		(at 70 81.5 0)
+		(layer "F.SilkS")
+		(effects
+			(font
+				(size 1 1)
+				(thickness 0.2)
+				(bold yes)
+			)
+		)
+	)
 	(gr_text "TRANSIMP."
 		(at 109.5 72.75 90)
@@
 			)
 		)
+	)
+	(gr_text "IN1"
+		(at 70 58.5 0)
+		(layer "F.SilkS")
+		(effects
+			(font
+				(size 1 1)
+				(thickness 0.2)
+				(bold yes)
+			)
+		)
