File: opto_elec_boards/phd_slave/phd_slave.kicad_sch (KiCad schematic)
At the start: 15 parts, among them J1 From Main Board, U1 TL082, U2 OPA551

Commit message: Update Opto Boards / To change : var +15V and var -15V ?
Connections:
- net +15V: no longer D4.1 (K), D5.1 (K)
- net GND: no longer J1.10 (Pin_10)
- new net RVAR_15V: D4.1 (K), D5.1 (K), J1.10 (Pin_10)
Other:
- moved on the sheet: D1, D2, D3, D4, D5, D6, R1, R2, R3, R4, R5, R6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
