File: opto_elec_boards/phd_slave_d25/phd_slave.kicad_sch (KiCad schematic)
At the start: 15 parts, among them J1 From Main Board, U1 TL082, U2 OPA551

Commit message: Update OptoBoard / D25 version
Parts:
- removed J1: From Main Board, Connector_PinSocket_2.54mm:PinSocket_2x10_P2.54mm_Horizontal, symbol Connector_Generic:Conn_02x10_Odd_Even
- added J13: FromMainBoard, Connector_Dsub:DSUB-25_Socket_Horizontal_P2.77x2.84mm_EdgePinOffset7.70mm_Housed_MountingHolesOffset9.12mm, symbol Connector:DB25_Socket_MountingHoles
Connections:
- net +15V: now also J13.4
- net -15V: now also J13.6; no longer D6.2 (A)
- net 3.3V: now also J13.14 (P14)
- net 5V: now also J13.1
- net GND: now also J13.0 (PAD), J13.16 (P16), J13.17 (P17), J13.18 (P18), J13.19 (P19), J13.20 (P20), J13.21 (P21), J13.22 (P22), J13.23 (P23), J13.5
- net IN1: now also J13.11
- net IN2: now also J13.12
- net OUT1: now also R6.1, U1.7, J13.10; no longer D4.2 (A), R4.1
- net OUT2: now also J13.9
- net OUT3: now also D4.2 (A), R4.1, J13.8; no longer R6.1, U1.7
- net OUT4: now also J13.7
- net RVAR_15V: now also D6.1 (K), J13.3
- net RVAR_3.3V: now also J13.15 (P15)
- net RVAR_5V: now also J13.2
- net SEL1: now also J13.13
- net SEL2: now also J13.25 (P25)
- net SEL3: now also J13.24 (P24)
- net at R6.2, U1.6 (-): now also D6.2 (A); no longer D6.1 (K)
Other:
- moved on the sheet: D6

Commit message: Update Opto Boards / Phd_slave_d25 with CT for transimpedance
Parts:
- added J1, J2: Conn_01x02, Connector_PinSocket_2.54mm:PinSocket_1x02_P2.54mm_Vertical, symbol Connector_Generic:Conn_01x02
Connections:
- net OUT1: now also J2.1 (Pin_1), J2.2 (Pin_2)
- net at D6.2 (A), R6.2, U1.6 (-): now also J1.1 (Pin_1), J1.2 (Pin_2)
Changed lines of the file:
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@@
 	)
 	(junction
+		(at 181.61 124.46)
+		(diameter 0)
+		(color 0 0 0 0)
+	)
+	(junction
 		(at 203.2 109.22)
 		(diameter 0)
@@
 	)
 	(junction
+		(at 203.2 124.46)
+		(diameter 0)
+		(color 0 0 0 0)
+	)
+	(junction
 		(at 101.6 35.56)
 		(diameter 0)
@@
 	)
 	(junction
+		(at 184.15 124.46)
+		(diameter 0)
+		(color 0 0 0 0)
+	)
+	(junction
 		(at 203.2 76.2)
 		(diameter 0)
@@
 	)
 	(junction
+		(at 200.66 124.46)
+		(diameter 0)
+		(color 0 0 0 0)
+	)
+	(junction
 		(at 157.48 73.66)
 		(diameter 0)
@@
 	(wire
 		(pts
+			(xy 200.66 124.46) (xy 200.66 130.81)
+		)
+		(stroke
+			(width 0)
+			(type default)
+		)
+	)
+	(wire
+		(pts
 			(xy 161.29 39.37) (xy 157.48 39.37)
 		)
@@
 	(wire
 		(pts
+			(xy 200.66 124.46) (xy 203.2 124.46)
+		)
+		(stroke
+			(width 0)
+			(type default)
+		)
+	)
+	(wire
+		(pts
 			(xy 129.54 96.52) (xy 130.81 96.52)
 		)
@@
 	(wire
 		(pts
+			(xy 184.15 124.46) (xy 184.15 130.81)
+		)
+		(stroke
+			(width 0)
+			(type default)
+		)
+	)
+	(wire
+		(pts
 			(xy 87.63 26.67) (xy 88.9 26.67)
 		)
@@
 	(wire
 		(pts
+			(xy 184.15 124.46) (xy 189.23 124.46)
+		)
+		(stroke
+			(width 0)
+			(type default)
+		)
+	)
+	(wire
+		(pts
 			(xy 157.48 71.12) (xy 157.48 73.66)
 		)
@@
 	(wire
 		(pts
-			(xy 181.61 124.46) (xy 189.23 124.46)
+			(xy 181.61 124.46) (xy 184.15 124.46)
 		)
 		(stroke
@@
 	(wire
 		(pts
+			(xy 203.2 124.46) (xy 203.2 130.81)
+		)
+		(stroke
+			(width 0)
+			(type default)
+		)
+	)
+	(wire
+		(pts
 			(xy 129.54 62.23) (xy 130.81 62.23)
 		)
@@
 	(wire
 		(pts
+			(xy 181.61 130.81) (xy 181.61 124.46)
+		)
+		(stroke
+			(width 0)
+			(type default)
+		)
+	)
+	(wire
+		(pts
 			(xy 241.3 82.55) (xy 243.84 82.55)
 		)
@@
 	(wire
 		(pts
-			(xy 196.85 124.46) (xy 203.2 124.46)
+			(xy 196.85 124.46) (xy 200.66 124.46)
 		)
 		(stroke
@@
 	)
 	(symbol
+		(lib_id "Connector_Generic:Conn_01x02")
+		(at 184.15 135.89 270)
+		(unit 1)
+		(exclude_from_sim no)
+		(in_bom yes)
+		(on_board yes)
+		(dnp no)
+		(fields_autoplaced yes)
+		(property "Reference" "J1"
+			(at 186.69 134.6199 90)
+			(effects
+				(font
+					(size 1.27 1.27)
+				)
+				(justify left)
+			)
+		)
+		(property "Value" "Conn_01x02"
+			(at 186.69 137.1599 90)
+			(effects
+				(font
+					(size 1.27 1.27)
+				)
+				(justify left)
+			)
+		)
+		(property "Footprint" "Connector_PinSocket_2.54mm:PinSocket_1x02_P2.54mm_Vertical"
+			(at 184.15 135.89 0)
+			(effects
+				(font
+					(size 1.27 1.27)
+				)
+				(hide yes)
+			)
+		)
+		(property "Datasheet" "~"
+			(at 184.15 135.89 0)
+			(effects
+				(font
+					(size 1.27 1.27)
+				)
+				(hide yes)
+			)
+		)
+		(property "Description" "Generic connector, single row, 01x02, script generated (kicad-library-utils/schlib/autogen/connector/)"
+			(at 184.15 135.89 0)
+			(effects
+				(font
+					(size 1.27 1.27)
+				)
+				(hide yes)
+			)
+		)
+		(pin "2"
+		)
+		(pin "1"
+		)
+		(instances
+			(project ""
+				(path "/57df33c0-6f05-4aba-b5b1-deb15b1b9db6"
+					(reference "J1")
+					(unit 1)
+				)
+			)
+		)
+	)
+	(symbol
 		(lib_id "power:GND")
 		(at 241.3 69.85 270)
@@
 					(unit 1)
 				)
+			)
+		)
+	)
+	(symbol
+		(lib_id "Connector_Generic:Conn_01x02")
+		(at 203.2 135.89 270)
+		(unit 1)
+		(exclude_from_sim no)
+		(in_bom yes)
+		(on_board yes)
+		(dnp no)
+		(fields_autoplaced yes)
+		(property "Reference" "J2"
+			(at 205.74 134.6199 90)
+			(effects
+				(font
+					(size 1.27 1.27)
+				)
+				(justify left)
+			)
+		)
+		(property "Value" "Conn_01x02"
+			(at 205.74 137.1599 90)
+			(effects
+				(font
+					(size 1.27 1.27)
+				)
+				(justify left)
+			)
+		)
+		(property "Footprint" "Connector_PinSocket_2.54mm:PinSocket_1x02_P2.54mm_Vertical"
+			(at 203.2 135.89 0)
+			(effects
+				(font
+					(size 1.27 1.27)
+				)
+				(hide yes)
+			)
+		)
+		(property "Datasheet" "~"
+			(at 203.2 135.89 0)
+			(effects
+				(font
+					(size 1.27 1.27)
+				)
+				(hide yes)
+			)
+		)
+		(property "Description" "Generic connector, single row, 01x02, script generated (kicad-library-utils/schlib/autogen/connector/)"
+			(at 203.2 135.89 0)
+			(effects
+				(font
+					(size 1.27 1.27)
+				)
+				(hide yes)
+			)
+		)
+		(pin "2"
+		)
+		(pin "1"
+		)
+		(instances
+			(project "phd_slave"
+				(path "/57df33c0-6f05-4aba-b5b1-deb15b1b9db6"
+					(reference "J2")
+					(unit 1)
+				)
